File: sketch_solar_weather_thingspeak/schematic/wemos_weather_station/wemos_weather_station.brd (EAGLE design)
At the start: 45.7 x 61.9 mm, 10 parts, among them U1 PHOTORESISTOR-5528-10K

Commit message: Schematic updated
Parts:
- moved BATTERY 53.9 mm to (3.81, 53.3), turned to 90 degrees
- moved SOLAR_PANEL 43.1 mm to (36.8, 66.0), turned to 270 degrees
- moved U$3 37.4 mm to (19.7, 53.2), turned to 180 degrees
- moved D1 31.0 mm to (29.2, 64.8), turned to 0 degrees
- moved C3 25.3 mm to (41.9, 77.3)
- moved U$2 22.3 mm to (20.5, 83.2)
- moved PROG_JUMPER 21.7 mm to (4.13, 91.6)
- moved U1 21.1 mm to (3.81, 83.4)
- moved U$1 11.7 mm to (40.6, 54.4), turned to 270 degrees
- moved C1 11.6 mm to (43.4, 62.0)
Routing:
- net GNDA: track 0.00 -> 73.6 mm
- net VCC: track 0.00 -> 62.0 mm
- net N$7: track 0.00 -> 51.1 mm
- net N$2: track 0.00 -> 26.2 mm
- net N$1: track 0.00 -> 12.1 mm
- net N$3: track 0.00 -> 7.77 mm
- net N$6: track 0.00 -> 7.58 mm
- net N$4: track 0.00 -> 7.57 mm
- net N$10: track 0.00 -> 5.04 mm
- net N$5: track 0.00 -> 2.54 mm

Commit message: schematic updated
Parts:
- added R1: 10k, resistor:0204/7
- moved U1 4.20 mm to (3.81, 79.2), turned to 270 degrees
- moved PROG_JUMPER 2.54 mm to (4.13, 89.0)
Connections:
- removed net GNDA: C1.2, C3.1, U$1.2, U$2.JP2.7, U$3.OUT-
- new net GND: C1.2, C3.1, R1.2, U$1.2, U$2.JP2.7, U$3.OUT-
- net N$11: now also R1.1
Routing:
- net GND: track 0.00 -> 82.9 mm
- net GNDA: track 73.6 -> 0.00 mm
- net N$11: track 0.00 -> 23.5 mm
- net N$6: track 7.58 -> 5.04 mm
- net N$10: track 5.04 -> 7.41 mm
Changed lines of the file:
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@@
 <attribute name="VALUE" x="27.178" y="61.976" size="1.27" layer="27" ratio="10"/>
 </element>
-<element name="PROG_JUMPER" library="pinhead" library_urn="urn:adsk.eagle:library:325" package="1X02" package3d_urn="urn:adsk.eagle:package:22435/2" value="" x="4.135" y="91.58" smashed="yes" rot="R90">
-<attribute name="NAME" x="2.3062" y="88.9638" size="1.27" layer="25" ratio="10" rot="R90"/>
-<attribute name="POPULARITY" value="98" x="75.255" y="116.98" size="1.778" layer="27" rot="R90" display="off"/>
-<attribute name="VALUE" x="7.31" y="89.04" size="1.27" layer="27" rot="R90"/>
+<element name="PROG_JUMPER" library="pinhead" library_urn="urn:adsk.eagle:library:325" package="1X02" package3d_urn="urn:adsk.eagle:package:22435/2" value="" x="4.135" y="89.04" smashed="yes" rot="R90">
+<attribute name="NAME" x="2.3062" y="86.4238" size="1.27" layer="25" ratio="10" rot="R90"/>
+<attribute name="POPULARITY" value="98" x="75.255" y="114.44" size="1.778" layer="27" rot="R90" display="off"/>
+<attribute name="VALUE" x="7.31" y="86.5" size="1.27" layer="27" rot="R90"/>
 </element>
 <element name="SOLAR_PANEL" library="pinhead" library_urn="urn:adsk.eagle:library:325" package="1X02" package3d_urn="urn:adsk.eagle:package:22435/2" value="" x="36.83" y="66.04" smashed="yes" rot="R270">
@@
 <attribute name="VALUE" x="19.735" y="63.4" size="1.27" layer="27" rot="R180" align="top-center"/>
 </element>
-<element name="U1" library="Seeed-Sensor" library_urn="urn:adsk.eagle:library:475" package="SNR2-3.0" package3d_urn="urn:adsk.eagle:package:32936/1" value="PHOTORESISTOR-5528-10K" x="3.81" y="83.38" smashed="yes" rot="R90">
-<attribute name="MPN" value="PHOTORESISTOR-5528-10K" x="68.58" y="111.32" size="1.778" layer="27" rot="R90" display="off"/>
-<attribute name="NAME" x="1.27" y="80.84" size="0.889" layer="25" ratio="11" rot="R90"/>
-<attribute name="VALUE" x="6.985" y="80.84" size="0.889" layer="27" ratio="11" rot="R90"/>
+<element name="U1" library="Seeed-Sensor" library_urn="urn:adsk.eagle:library:475" package="SNR2-3.0" package3d_urn="urn:adsk.eagle:package:32936/1" value="PHOTORESISTOR-5528-10K" x="3.81" y="79.18" smashed="yes" rot="R270">
+<attribute name="MPN" value="PHOTORESISTOR-5528-10K" x="-60.96" y="51.24" size="1.778" layer="27" rot="R270" display="off"/>
+<attribute name="NAME" x="6.35" y="81.72" size="0.889" layer="25" ratio="11" rot="R270"/>
+<attribute name="VALUE" x="0.635" y="81.72" size="0.889" layer="27" ratio="11" rot="R270"/>
+</element>
+<element name="R1" library="resistor" library_urn="urn:adsk.eagle:library:348" package="0204/7" package3d_urn="urn:adsk.eagle:package:25945/1" value="10k" x="4.045" y="68.445" smashed="yes" rot="R270">
+<attribute name="NAME" x="5.3404" y="70.985" size="0.9906" layer="25" ratio="10" rot="R270"/>
+<attribute name="VALUE" x="3.5624" y="70.0706" size="0.9906" layer="27" ratio="10" rot="R270"/>
 </element>
 </elements>
@@
 <contactref element="U$2" pad="JP2.4"/>
 <contactref element="U$1" pad="4"/>
-<wire x1="36.83" y1="59.49" x2="31.95" y2="85.14" width="0" layer="19" extent="1-1"/>
+<wire x1="31.95" y1="85.14" x2="36.83" y2="59.49" width="0" layer="19" extent="1-1"/>
 </signal>
 <signal name="N$9">
 <contactref element="U$1" pad="3"/>
 <contactref element="U$2" pad="JP2.3"/>
-<wire x1="39.37" y1="59.49" x2="31.95" y2="87.68" width="0" layer="19" extent="1-1"/>
+<wire x1="31.95" y1="87.68" x2="39.37" y2="59.49" width="0" layer="19" extent="1-1"/>
 </signal>
-<signal name="GNDA">
+<signal name="GND">
 <contactref element="U$3" pad="OUT-"/>
 <contactref element="U$1" pad="2"/>
@@
 <wire x1="11.7" y1="59.67" x2="8.94" y2="59.67" width="2" layer="16"/>
 <wire x1="8.94" y1="59.67" x2="8.94" y2="60.225" width="2" layer="16"/>
+<contactref element="R1" pad="2"/>
+<wire x1="8.94" y1="60.225" x2="4.045" y2="60.225" width="2" layer="16"/>
+<wire x1="4.045" y1="60.225" x2="4.045" y2="64.635" width="2" layer="16"/>
 <wire x1="41.91" y1="79.81" x2="42.705" y2="77.805" width="0" layer="19" extent="16-16"/>
 <wire x1="41.91" y1="59.49" x2="42.11" y2="62.02" width="0" layer="19" extent="1-1"/>
@@
 <wire x1="31.95" y1="74.98" x2="16.58" y2="74.98" width="2" layer="16"/>
 <wire x1="16.58" y1="74.98" x2="16.58" y2="46.215" width="2" layer="16"/>
+<wire x1="16.58" y1="55.88" x2="16.58" y2="46.215" width="0" layer="19" extent="1-16"/>
 <wire x1="16.58" y1="46.215" x2="8.94" y2="46.215" width="2" layer="16"/>
 <wire x1="8.94" y1="46.215" x2="8.94" y2="46.255" width="2" layer="16"/>
-<wire x1="31.95" y1="74.98" x2="3.81" y2="81.729" width="0" layer="19" extent="1-1"/>
+<wire x1="16.58" y1="55.88" x2="3.81" y2="80.831" width="0" layer="19" extent="1-1"/>
 </signal>
 <signal name="N$5">
@@
 <contactref element="PROG_JUMPER" pad="1"/>
 <wire x1="9.09" y1="87.68" x2="4.135" y2="87.68" width="2" layer="16"/>
-<wire x1="4.135" y1="87.68" x2="4.135" y2="90.31" width="2" layer="16"/>
+<wire x1="4.135" y1="87.68" x2="4.135" y2="87.77" width="2" layer="16"/>
 </signal>
 <signal name="N$10">
@@
 <contactref element="U$2" pad="JP1.1"/>
 <wire x1="9.09" y1="92.76" x2="4.135" y2="92.76" width="2" layer="16"/>
-<wire x1="4.135" y1="92.76" x2="4.135" y2="92.85" width="2" layer="16"/>
+<wire x1="4.135" y1="92.76" x2="4.135" y2="90.31" width="2" layer="16"/>
 </signal>
 <signal name="N$11">
 <contactref element="U1" pad="2"/>
 <contactref element="U$2" pad="JP1.2"/>
-<wire x1="3.81" y1="85.031" x2="9.09" y2="90.22" width="0" layer="19" extent="1-1"/>
+<contactref element="R1" pad="1"/>
+<wire x1="4.045" y1="72.255" x2="3.81" y2="72.255" width="2" layer="16"/>
+<wire x1="3.81" y1="72.255" x2="3.81" y2="77.529" width="2" layer="16"/>
+<wire x1="3.81" y1="77.529" x2="3.81" y2="78.8785" width="2" layer="1"/>
+<wire x1="7.0146" y1="90.09" x2="7.02" y2="90.09" width="2" layer="1"/>
+<wire x1="3.81" y1="78.8785" x2="7.0146" y2="78.8785" width="2" layer="1"/>
+<wire x1="7.0146" y1="78.8785" x2="7.0146" y2="90.09" width="2" layer="1"/>
+<wire x1="9.09" y1="90.22" x2="9.09" y2="90.09" width="2" layer="1"/>
+<wire x1="9.09" y1="90.09" x2="7.02" y2="90.09" width="2" layer="1"/>
 </signal>
 </signals>
